File: esp32_plus.sch (EAGLE design)
At the start: 27 parts, among them U1 ESP32 DEVKIT-V4

Commit message: Add files via upload
Parts:
- B, D: device jumper:JP1E -> jumper_edit:JP2E
- L1: SPICEPREFIX (none) -> L
- R1, R2, R3, R4, R5, R6: device rcl_Edit:R-EU_0207/7 -> rcl_Edit:R-EU_0207/10
Connections:
- net 3V3: now also D.3; no longer D.2
- net N$1: now also D.2; no longer D.1
